File: docs/hc-sr04-schematics/hc-sr04-schematics.kicad_sch (KiCad schematic)
At the start: 1 part

Commit message: docs
Parts:
- added R1: 330, symbol Device:R
- added R2: 470, symbol Device:R
- added U1: HC-SR04, XCVR_HC-SR04, symbol HC-SR04:HC-SR04
- gave numbers to parts that had none: 1
Connections:
- net at J1.12 (GPIO18/PWM0): now also U1.2 (TRIG)
- net at J1.18 (GPIO24): now also R1.2, R2.2
- net at J1.2 (5V): now also U1.1 (VCC)
- net at J1.6 (GND): now also R2.1, U1.4 (GND)
- new net: R1.1, U1.3 (ECHO)
- no-connect marks 0 -> 36
Changed lines of the file:
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@@
 (kicad_sch (version 20211123) (generator eeschema)
   (paper "A4")
+  (junction (at 104.14 94.488) (diameter 0) (color 0 0 0 0)
+  )
+  (junction (at 82.423 91.186) (diameter 0) (color 0 0 0 0)
+  )
+  (no_connect (at 144.653 117.348))
+  (no_connect (at 142.113 117.348))
+  (no_connect (at 162.433 64.008))
+  (no_connect (at 137.033 117.348))
+  (no_connect (at 139.573 117.348))
+  (no_connect (at 134.493 117.348))
+  (no_connect (at 121.793 99.568))
+  (no_connect (at 121.793 102.108))
+  (no_connect (at 121.793 97.028))
+  (no_connect (at 121.793 71.628))
+  (no_connect (at 121.793 69.088))
+  (no_connect (at 121.793 89.408))
+  (no_connect (at 121.793 91.948))
+  (no_connect (at 121.793 84.328))
+  (no_connect (at 121.793 81.788))
+  (no_connect (at 121.793 79.248))
+  (no_connect (at 162.433 71.628))
+  (no_connect (at 162.433 69.088))
+  (no_connect (at 162.433 61.468))
+  (no_connect (at 162.433 76.708))
+  (no_connect (at 162.433 79.248))
+  (no_connect (at 139.573 51.308))
+  (no_connect (at 144.653 51.308))
+  (no_connect (at 147.193 51.308))
+  (no_connect (at 121.793 61.468))
+  (no_connect (at 121.793 64.008))
+  (no_connect (at 162.433 102.108))
+  (no_connect (at 162.433 97.028))
+  (no_connect (at 162.433 104.648))
+  (no_connect (at 162.433 91.948))
+  (no_connect (at 162.433 94.488))
+  (no_connect (at 162.433 89.408))
+  (no_connect (at 162.433 86.868))
+  (no_connect (at 162.433 81.788))
+  (no_connect (at 149.733 117.348))
+  (no_connect (at 147.193 117.348))
+  (wire (pts (xy 104.14 94.488) (xy 121.793 94.488))
+    (stroke (width 0) (type default) (color 0 0 0 0))
+  )
+  (wire (pts (xy 82.423 91.186) (xy 82.423 75.565))
+    (stroke (width 0) (type default) (color 0 0 0 0))
+  )
+  (wire (pts (xy 101.6 91.186) (xy 101.6 94.488))
+    (stroke (width 0) (type default) (color 0 0 0 0))
+  )
+  (wire (pts (xy 101.6 94.488) (xy 104.14 94.488))
+    (stroke (width 0) (type default) (color 0 0 0 0))
+  )
+  (wire (pts (xy 104.14 78.359) (xy 104.14 82.042))
+    (stroke (width 0) (type default) (color 0 0 0 0))
+  )
+  (wire (pts (xy 82.423 117.348) (xy 82.423 91.186))
+    (stroke (width 0) (type default) (color 0 0 0 0))
+  )
+  (wire (pts (xy 104.14 94.488) (xy 104.14 89.662))
+    (stroke (width 0) (type default) (color 0 0 0 0))
+  )
+  (wire (pts (xy 137.033 51.308) (xy 82.423 51.308))
+    (stroke (width 0) (type default) (color 0 0 0 0))
+  )
+  (wire (pts (xy 96.393 70.485) (xy 82.423 70.485))
+    (stroke (width 0) (type default) (color 0 0 0 0))
+  )
+  (wire (pts (xy 131.953 117.348) (xy 82.423 117.348))
+    (stroke (width 0) (type default) (color 0 0 0 0))
+  )
+  (wire (pts (xy 83.566 78.359) (xy 83.566 73.025))
+    (stroke (width 0) (type default) (color 0 0 0 0))
+  )
+  (wire (pts (xy 96.52 91.186) (xy 101.6 91.186))
+    (stroke (width 0) (type default) (color 0 0 0 0))
+  )
+  (wire (pts (xy 83.566 73.025) (xy 82.423 73.025))
+    (stroke (width 0) (type default) (color 0 0 0 0))
+  )
+  (wire (pts (xy 82.423 91.186) (xy 88.9 91.186))
+    (stroke (width 0) (type default) (color 0 0 0 0))
+  )
+  (wire (pts (xy 82.423 51.308) (xy 82.423 67.945))
+    (stroke (width 0) (type default) (color 0 0 0 0))
+  )
+  (wire (pts (xy 104.14 78.359) (xy 83.566 78.359))
+    (stroke (width 0) (type default) (color 0 0 0 0))
+  )
+  (wire (pts (xy 121.793 74.168) (xy 96.393 74.168))
+    (stroke (width 0) (type default) (color 0 0 0 0))
+  )
+  (wire (pts (xy 96.393 74.168) (xy 96.393 70.485))
+    (stroke (width 0) (type default) (color 0 0 0 0))
+  )
   (symbol (lib_id "Connector:Raspberry_Pi_2_3") (at 142.113 84.328 0) (unit 1)
     (in_bom yes) (on_board yes) (fields_autoplaced)
-    (property "Reference" "J?" (id 0) (at 149.2124 48.26 0)
+    (property "Reference" "J1" (id 0) (at 149.2124 48.26 0)
       (effects (font (size 1.27 1.27)) (justify left))
     )
@@
     (pin "9")
   )
+  (symbol (lib_id "Device:R") (at 92.71 91.186 90) (unit 1)
+    (in_bom yes) (on_board yes) (fields_autoplaced)
+    (property "Reference" "R2" (id 0) (at 92.71 85.09 90))
+    (property "Value" "470" (id 1) (at 92.71 87.63 90))
+    (property "Footprint" "" (id 2) (at 92.71 92.964 90)
+      (effects (font (size 1.27 1.27)) hide)
+    )
+    (property "Datasheet" "~" (id 3) (at 92.71 91.186 0)
+      (effects (font (size 1.27 1.27)) hide)
+    )
+    (pin "1")
+    (pin "2")
+  )
+  (symbol (lib_id "Device:R") (at 104.14 85.852 0) (unit 1)
+    (in_bom yes) (on_board yes) (fields_autoplaced)
+    (property "Reference" "R1" (id 0) (at 106.68 84.5819 0)
+      (effects (font (size 1.27 1.27)) (justify left))
+    )
+    (property "Value" "330" (id 1) (at 106.68 87.1219 0)
+      (effects (font (size 1.27 1.27)) (justify left))
+    )
+    (property "Footprint" "" (id 2) (at 102.362 85.852 90)
+      (effects (font (size 1.27 1.27)) hide)
+    )
+    (property "Datasheet" "~" (id 3) (at 104.14 85.852 0)
+      (effects (font (size 1.27 1.27)) hide)
+    )
+    (pin "1")
+    (pin "2")
+  )
+  (symbol (lib_id "HC-SR04:HC-SR04") (at 77.343 70.485 0) (mirror y) (unit 1)
+    (in_bom yes) (on_board yes) (fields_autoplaced)
+    (property "Reference" "U1" (id 0) (at 72.263 60.198 0))
+    (property "Value" "HC-SR04" (id 1) (at 72.263 62.738 0))
+    (property "Footprint" "XCVR_HC-SR04" (id 2) (at 77.343 70.485 0)
+      (effects (font (size 1.27 1.27)) (justify bottom) hide)
+    )
+    (property "Datasheet" "" (id 3) (at 77.343 70.485 0)
+      (effects (font (size 1.27 1.27)) hide)
+    )
+    (property "MANUFACTURER" "Osepp" (id 4) (at 77.343 70.485 0)
+      (effects (font (size 1.27 1.27)) (justify bottom) hide)
+    )
+    (pin "1")
+    (pin "2")
+    (pin "3")
+    (pin "4")
+  )
   (sheet_instances
     (path "/" (page "1"))
@@
   (symbol_instances
     (path "/12c9f3e1-9431-42f8-b6f8-fb6fd35fc1cb"
-      (reference "J?") (unit 1) (value "Raspberry") (footprint "")
-    )
-  )
+      (reference "J1") (unit 1) (value "Raspberry") (footprint "")
+    )
+    (path "/77fb0648-035d-4c80-8793-b35373c65cc1"
+      (reference "R1") (unit 1) (value "330") (footprint "")
+    )
+    (path "/667eeaa2-f9d6-4b7d-8201-3cd5028933c9"
+      (reference "R2") (unit 1) (value "470") (footprint "")
+    )
+    (path "/be328f0a-6e1c-456b-9181-efb828298971"
+      (reference "U1") (unit 1) (value "HC-SR04") (footprint "XCVR_HC-SR04")
+    )
+  )
